Commit message: Added adjustable camera mount

File: openarm_bimanual_description/urdf/openarm_bimanual.urdf.xacro (robot description, xacro)
@@ -22,4 +22,5 @@
   <xacro:include filename="$(find openarm_description)/urdf/openarm.robot.xacro"/>
   <xacro:include filename="$(find openarm_bimanual_description)/urdf/openarm_pedestal.urdf"/>
+  <xacro:include filename="openarm_bimanual_cameraMount.xacro"/>
   <xacro:include filename="openarm_bimanual_sensors.xacro"/>
   <link name="world"/>

File: openarm_bimanual_description/urdf/openarm_bimanual_cameraMount.xacro (robot description, xacro)
@@ -13,8 +13,5 @@
 -->
 <robot xmlns:xacro="http://www.ros.org/wiki/xacro">
-    <xacro:include filename="$(find realsense2_description)/urdf/_d435i.urdf.xacro"/>
     <xacro:include filename="$(find camAssembly_4H_description)/urdf/camAssembly_4H.urdf.xacro"/>
-    <xacro:sensor_d435i parent="camAttachment_1" use_nominal_extrinsics="true">
-        <origin xyz="0.015 -0.045 0.0" rpy="0 0 0"/>
-    </xacro:sensor_d435i>
+    <xacro:cam_mount parent="pedestal_link"/>
 </robot>
