Commit message: Add camera mount to robot description xacros

File: openarm_bimanual_description/urdf/camera_mount.urdf.xacro (robot description, xacro)
@@ -2,7 +2,4 @@
 <robot name="camAssembly_4H" xmlns:xacro="http://www.ros.org/wiki/xacro">
   <xacro:macro name="cam_mount" params="parent">
-    <xacro:include filename="$(find camAssembly_4H_description)/urdf/materials.xacro" />
-    <xacro:include filename="$(find camAssembly_4H_description)/urdf/camAssembly_4H.trans" />
-    <xacro:include filename="$(find camAssembly_4H_description)/urdf/camAssembly_4H.gazebo" />
     <link name="cam_4h_base_link">
       <inertial>
@@ -14,12 +11,12 @@
         <origin xyz="0 0 0" rpy="0 0 0"/>
         <geometry>
-          <mesh filename="file://$(find camAssembly_4H_description)/meshes/base_link.stl" scale="0.001 0.001 0.001"/>
+          <mesh filename="file://$(find openarm_bimanual_description)/meshes/base_link.stl" scale="0.001 0.001 0.001"/>
         </geometry>
-        <material name="silver"/>
+        <material name="gray"/>
       </visual>
       <collision>
         <origin xyz="0 0 0" rpy="0 0 0"/>
         <geometry>
-          <mesh filename="file://$(find camAssembly_4H_description)/meshes/base_link.stl" scale="0.001 0.001 0.001"/>
+          <mesh filename="file://$(find openarm_bimanual_description)/meshes/base_link.stl" scale="0.001 0.001 0.001"/>
         </geometry>
       </collision>
@@ -34,12 +31,12 @@
         <origin xyz="0.015756 -0.045243 -0.004" rpy="0 0 0"/>
         <geometry>
-          <mesh filename="file://$(find camAssembly_4H_description)/meshes/camAttachment_1.stl" scale="0.001 0.001 0.001"/>
+          <mesh filename="file://$(find openarm_bimanual_description)/meshes/camAttachment_1.stl" scale="0.001 0.001 0.001"/>
         </geometry>
-        <material name="silver"/>
+        <material name="gray"/>
       </visual>
       <collision>
         <origin xyz="0.015756 -0.045243 -0.004" rpy="0 0 0"/>
         <geometry>
-          <mesh filename="file://$(find camAssembly_4H_description)/meshes/camAttachment_1.stl" scale="0.001 0.001 0.001"/>
+          <mesh filename="file://$(find openarm_bimanual_description)/meshes/camAttachment_1.stl" scale="0.001 0.001 0.001"/>
         </geometry>
       </collision>

File: openarm_bimanual_description/urdf/openarm_bimanual.urdf.xacro (robot description, xacro)
@@ -22,6 +22,5 @@
   <xacro:include filename="$(find openarm_description)/urdf/openarm.robot.xacro"/>
   <xacro:include filename="$(find openarm_bimanual_description)/urdf/openarm_pedestal.urdf"/>
-  <xacro:include filename="openarm_bimanual_cameraMount.xacro"/>
-  <xacro:include filename="openarm_bimanual_sensors.xacro"/>
+  <xacro:include filename="$(find openarm_bimanual_description)/urdf/openarm_sensors.urdf.xacro"/>
   <link name="world"/>
   <joint name="dummy_joint" type="fixed">

File: openarm_bimanual_description/urdf/openarm_sensors.urdf.xacro (robot description, xacro)
@@ -14,5 +14,6 @@
 <robot xmlns:xacro="http://www.ros.org/wiki/xacro">
     <xacro:include filename="$(find realsense2_description)/urdf/_d435i.urdf.xacro"/>
-    <xacro:include filename="$(find camAssembly_4H_description)/urdf/camAssembly_4H.urdf.xacro"/>
+    <xacro:include filename="$(find openarm_bimanual_description)/urdf/camera_mount.urdf.xacro"/>
+    <xacro:cam_mount parent="pedestal_link"/>
     <xacro:sensor_d435i parent="camAttachment_1" use_nominal_extrinsics="true">
         <origin xyz="0.015 -0.045 0.0" rpy="0 0 0"/>

Commit message: Change from rev joint to fixed with presets

File: openarm_bimanual_description/urdf/camera_mount.urdf.xacro (robot description, xacro)
@@ -1,5 +1,6 @@
 <?xml version="1.0" ?>
 <robot name="camAssembly_4H" xmlns:xacro="http://www.ros.org/wiki/xacro">
-  <xacro:macro name="cam_mount" params="parent">
+  <xacro:macro name="cam_mount" params="parent cam_angle:=0.785">
+    <!-- cam_angle options: 0.401 (straight), 0.785 (mid), 1.186 (max tilt) -->
     <link name="cam_4h_base_link">
       <inertial>
@@ -42,10 +43,8 @@
       </collision>
     </link>
-    <joint name="cam_rev_joint" type="revolute">
-      <origin xyz="-0.015756 0.045243 0.004" rpy="0 0 0"/>
+    <joint name="cam_fixed_joint" type="fixed">
+      <origin xyz="-0.015756 0.045243 0.004" rpy="0 ${cam_angle} 0"/>
       <parent link="cam_4h_base_link"/>
       <child link="camAttachment_1"/>
-      <axis xyz="0 1 0"/>
-      <limit lower="0" upper="1.186" effort="1.0" velocity="1.0"/>
     </joint>
     <joint name="cam_mount_joint" type="fixed">

File: openarm_bimanual_description/urdf/openarm_sensors.urdf.xacro (robot description, xacro)
@@ -15,5 +15,6 @@
     <xacro:include filename="$(find realsense2_description)/urdf/_d435i.urdf.xacro"/>
     <xacro:include filename="$(find openarm_bimanual_description)/urdf/camera_mount.urdf.xacro"/>
-    <xacro:cam_mount parent="pedestal_link"/>
+    <!-- pass tilt angle, presets are 0.000, 0.401, 0.785, 1.186 -->
+    <xacro:cam_mount parent="pedestal_link" cam_angle="0.000"/>
     <xacro:sensor_d435i parent="camAttachment_1" use_nominal_extrinsics="true">
         <origin xyz="0.015 -0.045 0.0" rpy="0 0 0"/>

Commit message: Fix syntax

File: openarm_bimanual_description/urdf/camera_mount.urdf.xacro (robot description, xacro)
@@ -1,6 +1,5 @@
 <?xml version="1.0" ?>
 <robot name="camAssembly_4H" xmlns:xacro="http://www.ros.org/wiki/xacro">
-  <xacro:macro name="cam_mount" params="parent cam_angle:=0.785">
-    <!-- cam_angle options: 0.401 (straight), 0.785 (mid), 1.186 (max tilt) -->
+  <xacro:macro name="cam_mount" params="parent:='' cam_angle:=''">
     <link name="cam_4h_base_link">
       <inertial>

File: openarm_bimanual_description/urdf/openarm_sensors.urdf.xacro (robot description, xacro)
@@ -15,6 +15,6 @@
     <xacro:include filename="$(find realsense2_description)/urdf/_d435i.urdf.xacro"/>
     <xacro:include filename="$(find openarm_bimanual_description)/urdf/camera_mount.urdf.xacro"/>
-    <!-- pass tilt angle, presets are 0.000, 0.401, 0.785, 1.186 -->
-    <xacro:cam_mount parent="pedestal_link" cam_angle="0.000"/>
+    <!-- pass tilt angle, presets are 0.401, 0.785, 1.186 -->
+    <xacro:cam_mount parent="pedestal_link" cam_angle="0.401"/>
     <xacro:sensor_d435i parent="camAttachment_1" use_nominal_extrinsics="true">
         <origin xyz="0.015 -0.045 0.0" rpy="0 0 0"/>
