Commit message: Configure mock and prefix

File: openarm_description/urdf/openarm.ros2_control.xacro (robot description, xacro)
@@ -13,13 +13,17 @@
 -->
 <robot xmlns:xacro="http://www.ros.org/wiki/xacro">
-    <xacro:macro name="openarm_ros2_control" params="name initial_positions_file prefix:='' can_device='can0'">
+    <xacro:macro name="openarm_ros2_control" params="name initial_positions_file prefix:='' can_device='can0' use_mock_hardware:=false mock_sensor_commands:=false">
         <xacro:property name="initial_positions" value="${xacro.load_yaml(initial_positions_file)['initial_positions']}"/>
         <ros2_control name="${prefix}${name}" type="system">
             <hardware>
-                <!-- By default, set up controllers for simulation. This won't work on real hardware -->
-                <!-- <plugin>mock_components/GenericSystem</plugin> -->
-                <plugin>openarm_hardware/OpenArmHW</plugin>
-                <param name="prefix">${prefix}</param>
-                <param name="can_device">${can_device}</param>
+                <xacro:if value="${use_mock_hardware}">
+                    <plugin>mock_components/GenericSystem</plugin>
+                    <param name="mock_sensor_commands">${mock_sensor_commands}</param>
+                </xacro:if>
+                <xacro:unless value="${use_mock_hardware}">
+                    <plugin>openarm_hardware/OpenArmHW</plugin>
+                    <param name="prefix">${prefix}</param>
+                    <param name="can_device">${can_device}</param>
+                </xacro:unless>
             </hardware>
             <joint name="${prefix}rev1">

File: openarm_description/urdf/openarm.urdf.xacro (robot description, xacro)
@@ -13,6 +13,9 @@
 -->
 <robot xmlns:xacro="http://www.ros.org/wiki/xacro" name="openarm">
+    <xacro:arg name="prefix" default="" />
+    <xacro:arg name="use_mock_hardware" default="false" />
+    <xacro:arg name="mock_sensor_commands" default="false" />
     <xacro:include filename="openarm.xacro"/>
-    <xacro:openarm/>
+    <xacro:openarm prefix="$(arg prefix)" use_mock_hardware="$(arg use_mock_hardware)" mock_sensor_commands="$(arg mock_sensor_commands)"/>
     <xacro:include filename="$(find openarm_description)/urdf/openarm_sensors.xacro"/>
 </robot>

File: openarm_description/urdf/openarm.xacro (robot description, xacro)
@@ -19,5 +19,5 @@
         <color rgba="${50/255} ${50/255} ${50/255} 1.0"/>
     </material>
-    <xacro:macro name="openarm" params="side:='right' prefix:='' zero_pos='up' can_device='can0'">
+    <xacro:macro name="openarm" params="side:='right' prefix:='' zero_pos='up' can_device='can0' use_mock_hardware:=false mock_sensor_commands:=false">
         <!-- side right, left -->
         <!-- recommended prefixes left_, right_, etc. -->
@@ -27,5 +27,5 @@
         <xacro:include filename="$(find openarm_description)/urdf/openarm.ros2_control.xacro" />
         <xacro:arg name="initial_positions_file" default="$(find openarm_description)/config/initial_positions.yaml" />
-        <xacro:openarm_ros2_control name="OpenArmHW" prefix="${prefix}" initial_positions_file="$(arg initial_positions_file)" can_device="${can_device}"/>
+        <xacro:openarm_ros2_control name="OpenArmHW" prefix="${prefix}" initial_positions_file="$(arg initial_positions_file)" can_device="${can_device}" use_mock_hardware="${use_mock_hardware}" mock_sensor_commands="${mock_sensor_commands}"/>
         <link name="${prefix}dummy_link"/>
         <joint name="${prefix}dummy_joint" type="fixed">

Commit message: Separate robot hw and control for urdf

File: openarm_description/urdf/openarm.ros2_control.xacro (robot description, xacro)
@@ -88,9 +88,4 @@
                 <state_interface name="velocity"/>
             </joint>
-            <!-- <joint name="${prefix}right_pris2">
-                <state_interface name="position">
-                  <param name="initial_value">${initial_positions['right_pris2']}</param>
-                </state_interface>
-            </joint> -->
         </ros2_control>
     </xacro:macro>

File: openarm_description/urdf/openarm.urdf.xacro (robot description, xacro)
@@ -13,9 +13,18 @@
 -->
 <robot xmlns:xacro="http://www.ros.org/wiki/xacro" name="openarm">
+    <!-- Robot description parameters -->
     <xacro:arg name="prefix" default="" />
+    <xacro:arg name="side" default="right" />
+    <xacro:arg name="zero_pos" default="up" />
+    <!-- Control-related parameters -->
+    <xacro:arg name="can_device" default="can0" />
     <xacro:arg name="use_mock_hardware" default="false" />
     <xacro:arg name="mock_sensor_commands" default="false" />
-    <xacro:include filename="openarm.xacro"/>
-    <xacro:openarm prefix="$(arg prefix)" use_mock_hardware="$(arg use_mock_hardware)" mock_sensor_commands="$(arg mock_sensor_commands)"/>
-    <xacro:include filename="$(find openarm_description)/urdf/openarm_sensors.xacro"/>
+    <!-- Include robot description (without control parameters) -->
+    <xacro:include filename="openarm.robot.xacro"/>
+    <xacro:openarm_robot prefix="$(arg prefix)" side="$(arg side)" zero_pos="$(arg zero_pos)"/>
+    <!-- Include control configuration (with only control parameters) -->
+    <xacro:include filename="$(find openarm_description)/urdf/openarm.ros2_control.xacro"/>
+    <xacro:arg name="initial_positions_file" default="$(find openarm_description)/config/initial_positions.yaml" />
+    <xacro:openarm_ros2_control name="OpenArmHW" prefix="$(arg prefix)" initial_positions_file="$(arg initial_positions_file)" can_device="$(arg can_device)" use_mock_hardware="$(arg use_mock_hardware)" mock_sensor_commands="$(arg mock_sensor_commands)"/>
 </robot>
