Commit message: refactor: separate robot and control xacros (#22)
The previous URDF directory structure used has a chained call from
**openarm.urdf.xacro** -> **openarm.xacro** ->
**openarm.ros2_control.xacro**.
**openarm.xacro** takes both robot hardware description and
control/communication configuration arguments but the file content is
only about robot description.

- Renamed **openarm.xacro** to **openarm.robot.xacro**. This file now
contains only the robot's hardware description, including links, joints,
visuals, and inertial properties.
- **openarm.control.xacro** handles all ROS 2 control configurations,
including hardware interfaces, joint interfaces, and CAN device setup.
- Updated openarm.urdf.xacro (entry point)Calls both
**openarm.robot.xacro** and **openarm.control.xacro**.

This change should separates responsibilities and arguments for each
subsystem.
Have tested with bringup scripts for both single-arm and bimanual
configurations.

Configure mock and prefix

File: openarm_description/urdf/openarm.robot.xacro (robot description, xacro)
@@ -19,5 +19,5 @@
         <color rgba="${50/255} ${50/255} ${50/255} 1.0"/>
     </material>
-    <xacro:macro name="openarm" params="side:='right' prefix:='' zero_pos='up' can_device='can0' use_mock_hardware:=false mock_sensor_commands:=false">
+    <xacro:macro name="openarm_robot" params="side:='right' prefix:='' zero_pos='up'">
         <!-- side right, left -->
         <!-- recommended prefixes left_, right_, etc. -->
@@ -25,7 +25,4 @@
         <xacro:property name="reflect" value="${1 if side=='right' else -1}"/>
         <xacro:property name="rotate" value="${0 if side=='right' else pi}"/>
-        <xacro:include filename="$(find openarm_description)/urdf/openarm.ros2_control.xacro" />
-        <xacro:arg name="initial_positions_file" default="$(find openarm_description)/config/initial_positions.yaml" />
-        <xacro:openarm_ros2_control name="OpenArmHW" prefix="${prefix}" initial_positions_file="$(arg initial_positions_file)" can_device="${can_device}" use_mock_hardware="${use_mock_hardware}" mock_sensor_commands="${mock_sensor_commands}"/>
         <link name="${prefix}dummy_link"/>
         <joint name="${prefix}dummy_joint" type="fixed">
